File: kicad_template/template.kicad_sch (KiCad schematic)
At the start: 0 parts

Commit message: update: 10 files changed, 1276 insertions(+), 597 deletions(-) (2026-07-31 13:40)
Connections:
- no-connect marks 1 -> 0
Other:
- title: KiCad Template Schematic -> (none)
Changed lines of the file:
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@@
-(kicad_sch (version 20230121) (generator eeschema)
-  (paper "A4")
-  (title_block
-    (title "KiCad Template Schematic")
-    (date "")
-    (rev "1.0")
-    (company "")
-  )
-  (no_connect (at 0 0))
-  (sheet_instances
-    (path "/" (page "1"))
-  )
+(kicad_sch
+	(version 20231120)
+	(generator "eeschema")
+	(generator_version "9.0")
+	(paper "A4")
+	(title_block
+		(title "")
+		(date "")
+		(rev "1.0")
+		(company "")
+	)
+	(sheet_instances
+		(path "/"
+			(page "1")
+		)
+	)
 )
